File: Hardware/hdmi.sch (KiCad schematic (older format))
At the start: 2 parts, among them U1 TS3DV642

Commit message: Designed layout for power stage and for control logic
Parts:
- added J11, J12, J13: HMDI, Custom:HDMI_SMD, symbol Custom:HMDI
- added R3, R4: 10K, Resistors_SMD:R_0805_HandSoldering, symbol device:R
- added R6, R7: 2k, Resistors_SMD:R_0805_HandSoldering, symbol device:R
- added R8: 100k, Resistors_SMD:R_0805_HandSoldering, symbol device:R
Connections:
- net labels added: +5V, CEC, CECA, CECB, CLK+, CLK-, CLKA+, CLKA-, CLKB+, CLKB-, D0+, D0-, D0A+, D0A-, D0B+, D0B-, D1+, D1-, D1A+, D1A-, D1B+, D1B-, D2+, D2-, D2A+, D2A-, D2B+, D2B-, HPD, HPDA, HPDB, SCL, SCLA, SCLB, SDA, SDAA, SDAB
- net labels removed: L_HI
- wire segments 3 -> 38
- no-connect marks 0 -> 3
Other:
- note added: "Channel A"
- note added: "Channel B"
- note added: "Convergence"
