File: Hardware/kvm.kicad_pcb (KiCad board)
At the start: 2 copper layers, 0 parts

Commit message: Designed layout for power stage and for control logic
Parts:
- added C1: 0.1uF, Capacitors_SMD:C_0805_HandSoldering, F.Cu at (182.0, 78.0)
- added C10: 0.1uF, Capacitors_SMD:C_0805_HandSoldering, F.Cu at (318.2, 104.9)
- added C2: 1uF, Capacitors_SMD:C_0805_HandSoldering, F.Cu at (184.0, 78.0)
- added C3: 4.7uF, Capacitors_SMD:C_0805_HandSoldering, F.Cu at (186.0, 78.0)
- added C4: 10uF, Capacitors_SMD:C_0805_HandSoldering, F.Cu at (173.0, 78.0)
- added C5: 1uF, Capacitors_SMD:C_0805_HandSoldering, F.Cu at (171.0, 78.0)
- added C6: 0.1uF, Capacitors_SMD:C_0805_HandSoldering, F.Cu at (169.0, 78.0)
- added C7: 0.1uF, Capacitors_SMD:C_0805_HandSoldering, F.Cu at (347.4, 113.8)
- added C8: 0.1uF, Capacitors_SMD:C_0805_HandSoldering, F.Cu at (313.3, 104.9)
- added C9: 0.1uF, Capacitors_SMD:C_0805_HandSoldering, F.Cu at (308.5, 104.9)
- added D1: LED, LEDs:LED_0805_HandSoldering, F.Cu at (190.8, 106.8)
- added J1: USB_A, Custom:USB_A_SMD, F.Cu at (141.8, 71.5)
- added J10: USB_B_Micro, Custom:micro_usb_smd, F.Cu at (193.2, 91.5)
- added J11: HMDI, Custom:HDMI_SMD, F.Cu at (83.8, 86.5)
- added J12: HMDI, Custom:HDMI_SMD, F.Cu at (83.8, 66.5)
- added J13: HMDI, Custom:HDMI_SMD, F.Cu at (83.8, 106.5)
- added J2: USB_A, Custom:USB_A_SMD, F.Cu at (-18.2, 106.5)
- added J3: USB_A, Custom:USB_A_SMD, F.Cu at (5.75, 150.6)
- added J4: USB_B, Custom:USB_B_SMD, F.Cu at (-24.8, 62.5)
- added J5: USB_B, Custom:USB_B_SMD, F.Cu at (-29.0, 128.5)
- added J6: USB_B, Custom:USB_B_SMD, F.Cu at (-9.75, 179.6)
- added J7: USB_B, Custom:USB_B_SMD, F.Cu at (-24.8, 81.0)
- added J8: USB_B, Custom:USB_B_SMD, F.Cu at (7.25, 102.0)
- added J9: USB_B, Custom:USB_B_SMD, F.Cu at (33.8, 167.6)
- added Q1: Q_NMOS_GSD, TO_SOT_Packages_SMD:SOT-23_Handsoldering, F.Cu at (186.5, 101.5)
- added R1: 1k, Resistors_SMD:R_0805_HandSoldering, F.Cu at (173.5, 99.0)
- added R2: 1k, Resistors_SMD:R_0805_HandSoldering, F.Cu at (173.5, 83.8)
- added R3: 10K, Resistors_SMD:R_0805_HandSoldering, F.Cu at (347.5, 119.2)
- added R4: 10K, Resistors_SMD:R_0805_HandSoldering, F.Cu at (352.3, 113.7)
- added R5: 220, Resistors_SMD:R_0805_HandSoldering, F.Cu at (190.8, 108.8)
- added R6: 2k, Resistors_SMD:R_0805_HandSoldering, F.Cu at (311.4, -6.09)
- added R7: 2k, Resistors_SMD:R_0805_HandSoldering, F.Cu at (316.6, -6.09)
- added R8: 100k, Resistors_SMD:R_0805_HandSoldering, F.Cu at (321.7, -6.09)
- added REF**: MountingHole_2.2mm_M2_Pad, Mounting_Holes:MountingHole_2.2mm_M2_Pad, F.Cu at (97.8, 113.5)
- added REF**: MountingHole_2.2mm_M2_Pad, Mounting_Holes:MountingHole_2.2mm_M2_Pad, F.Cu at (97.8, 69.5)
- added REF**: MountingHole_2.2mm_M2_Pad, Mounting_Holes:MountingHole_2.2mm_M2_Pad, F.Cu at (191.8, 113.5)
- added REF**: MountingHole_2.2mm_M2_Pad, Mounting_Holes:MountingHole_2.2mm_M2_Pad, F.Cu at (191.8, 69.5)
- added SW1: SW_DIP_x01, Custom:TL3342F160_tact_switch, F.Cu at (176.9, 97.6)
- added SW2: SW_DIP_x01, Custom:TL3342F160_tact_switch, F.Cu at (183.2, 85.3)
- added SW3: SW_DPDT_x2, Custom:GH39P0, F.Cu at (190.8, 84.0)
- added SW4: SW_DIP_x01, Custom:TL3342F160_tact_switch, F.Cu at (189.5, 104.3)
- added TP1: Test_Point, Custom:1.5mm_test_point, F.Cu at (186.0, 84.8)
- added TP2: Test_Point, Custom:1.5mm_test_point, F.Cu at (186.2, 72.8)
- added TP3: Test_Point, Custom:1.5mm_test_point, F.Cu at (172.2, 72.8)
- added U1: TS3DV642, Custom:WQFN42, F.Cu at (90.0, 83.6)
- added U2: SPX1117, TO_SOT_Packages_SMD:SOT-223-3_TabPin2, F.Cu at (177.5, 76.0)
- added U3: Double NAND, Custom:VSSOP8_2.4x2.1mm_Pitch0.5mm, F.Cu at (183.0, 91.5)
- added U4: TS3USB3031, Custom:WQGN12, F.Cu at (-17.8, 69.5)
- added U5: TS3USB3031, Custom:WQGN12, F.Cu at (-7.95, 123.5)
- added U6: TS3USB3031, Custom:WQGN12, F.Cu at (12.2, 168.1)
Routing:
- net VCC: track 0.00 -> 56.6 mm
- net GND: track 0.00 -> 45.8 mm
- net Net-(R5-Pad1): track 0.00 -> 17.8 mm
- net CTRL: track 0.00 -> 16.9 mm
- net +5VA: track 0.00 -> 15.4 mm
- net +5V: track 0.00 -> 11.0 mm
- net Net-(R1-Pad1): track 0.00 -> 8.51 mm
- net Net-(R2-Pad2): track 0.00 -> 8.11 mm
- net Net-(D1-Pad1): track 0.00 -> 5.69 mm
- net +5VD: track 0.00 -> 5.22 mm
- net Net-(D1-Pad2): track 0.00 -> 2.00 mm
- net Net-(U3-Pad2): track 0.00 -> 0.50 mm
Other:
- board outline added: 100 x 50 mm
- net class Default: clearance 0.1524 -> 0.2032; trace_width 0.1524 -> 0.254
- rule trace_clearance: 0.1524 -> 0.2032
- board text added: "A"
- board text added: "B"
