File: Hardware/kvm.sch (KiCad schematic (older format))
At the start: 13 parts, among them J10 USB_B_Micro, SW1 SW_DIP_x01, SW2 SW_DIP_x01, U2 SPX1117, U3 Double NAND

Commit message: Designed layout for power stage and for control logic
Parts:
- added D1: LED, LEDs:LED_0805_HandSoldering, symbol device:LED
- added Q1: Q_NMOS_GSD, TO_SOT_Packages_SMD:SOT-23_Handsoldering, symbol device:Q_NMOS_GSD
- added R5: 220, Resistors_SMD:R_0805_HandSoldering, symbol device:R
- added SW3: SW_DPDT_x2, Custom:GH39P0, symbol Switch:SW_DPDT_x2
- added SW4: SW_DIP_x01, Custom:TL3342F160_tact_switch, symbol Switch:SW_DIP_x01
- added TP1, TP2, TP3: Test_Point, Custom:1.5mm_test_point, symbol Connector:Test_Point
- SW1, SW2: footprint (none) -> Custom:TL3342F160_tact_switch
Connections:
- net labels added: +5VA, +5VD
- wire segments 51 -> 61
