File: Hardware/usb.sch (KiCad schematic (older format))
At the start: 12 parts, among them J1 USB_A, J2 USB_A, J3 USB_A, J4 USB_B, J5 USB_B, J6 USB_B, J7 USB_B, J8 USB_B, J9 USB_B, U4 TS3USB30EDGSR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

Commit message: Designed layout for power stage and for control logic
Parts:
- removed U4, U5, U6: TS3USB30EDGSR, Custom:MSOP10_3x3mm_Pitch0.5mm, symbol Custom:TS3USB30EDGSR
- added C10, C8, C9: 0.1uF, Capacitors_SMD:C_0805_HandSoldering, symbol device:C
- added U4, U5, U6: TS3USB3031, Custom:WQGN12, symbol Custom:TS3USB3031
- J4, J5, J6, J7, J8, J9: footprint (none) -> Custom:USB_B_SMD
Connections:
- net labels added: +5VD
- net labels removed: +5V
- wire segments 51 -> 61
- no-connect marks 6 -> 12

Commit message: USB ports and USB muxes to change
Parts:
- removed C10, C9: 0.1uF, Capacitors_SMD:C_0805_HandSoldering, symbol device:C
- removed J4, J5, J6, J7, J8, J9: USB_B, Custom:USB_B_SMD, symbol Connector:USB_B
- removed U4, U5, U6: TS3USB3031, Custom:WQGN12, symbol Custom:TS3USB3031
- added C? (x2): 0.1uF, Capacitors_SMD:C_0805_HandSoldering, symbol device:C
- added U? (x3): TS3USB3000, symbol Custom:TS3USB3000
Connections:
- wire segments 61 -> 40
- no-connect marks 12 -> 0
